File: Hardware/devboard Rev1.1/ESP32MP3-dev-board.kicad_pcb (KiCad board)
At the start: 2 copper layers, 42 x 70 mm, 64 parts, among them J1 USB_C_Receptacle_USB2.0_16P, J2 Micro_SD_Card_Det1, Q1 SS8050, Q2 SS8050, SW1 SW_SPDT, SW2 EN, SW3 BOOT, SW4 LEFT, SW5 UP, SW6 ENTER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

Commit message: fixed switch footprint and changed buttons pins to avoid bootstrapping pins
Connections:
- SW4 pad 2: /Buttons/BTN LEFT -> unconnected-(SW4-Pad2)
- SW5 pad 2: /Buttons/BTN UP -> unconnected-(SW5-Pad2)
- SW6 pad 2: /Buttons/BTN ENTER -> unconnected-(SW6-Pad2)
- SW7 pad 2: /Buttons/BTN DOWN -> unconnected-(SW7-Pad2)
- SW8 pad 2: /Buttons/BTN RIGHT -> unconnected-(SW8-Pad2)
- U3 pad 24: /Buttons/BTN ENTER -> unconnected-(U3-IO2-Pad24)
- U3 pad 26: /Buttons/BTN LEFT -> /Buttons/BTN ENTER
- U3 pad 28: /Buttons/BTN DOWN -> /Buttons/BTN LEFT
- U3 pad 29: unconnected-(U3-IO5-Pad29) -> /Buttons/BTN DOWN
Routing:
- net /Buttons/BTN ENTER: track 27.7 -> 33.8 mm
- net /Buttons/BTN RIGHT: track 24.7 -> 20.7 mm
- net /Buttons/BTN DOWN: track 39.3 -> 36.4 mm
- net /Buttons/BTN LEFT: track 30.3 -> 28.3 mm
- net /MCU/µSD CS: track 19.9 -> 21.7 mm
